Commit message: updating

File: fws_description/gazebo/fws_robot.gazebo.xacro (robot description, xacro)
@@ -38,6 +38,41 @@
           <frame_id>/lidar_head_link</frame_id>
         </lidar>
-        <alwaysOn>ture</alwaysOn>
+        <alwaysOn>true</alwaysOn>
         <visualize>true</visualize>
+      </sensor>
+    </gazebo>
+    <!-- GPS Link and Joint -->
+    <link name="gps_link">
+      <visual>
+        <geometry>
+          <sphere radius="0.01"/>
+        </geometry>
+        <material name="white"/>
+      </visual>
+    </link>
+    <joint name="gps_joint" type="fixed">
+      <parent link="base_link"/>
+      <child link="gps_link"/>
+      <origin xyz="0 0 0.1" rpy="0 0 0"/>
+    </joint>
+    <!-- GPS Sensor Plugin -->
+    <gazebo reference="gps_link">
+      <sensor name="gps_sensor" type="navsat">
+        <pose>0 0 0 0 0 0</pose>
+        <update_rate>5.0</update_rate>
+        <navsat>
+          <horizontal>
+            <noise type="gaussian">
+              <mean>0</mean>
+              <stddev>1e-6</stddev>
+            </noise>
+          </horizontal>
+          <vertical>
+            <noise type="gaussian">
+              <mean>0</mean>
+              <stddev>1e-6</stddev>
+            </noise>
+          </vertical>
+        </navsat>
       </sensor>
     </gazebo>

File: fws_description/robots/fws_robot.urdf.xacro (robot description, xacro)
@@ -91,3 +91,11 @@
   <xacro:fws_robot_gazebo/>
   <xacro:fws_robot_ros2_control/>
+  <!-- <gazebo>
+  <plugin name="gz::sim::systems::PosePublisher" filename="gz-sim-pose-publisher-system">
+      <publish_link_pose>true</publish_link_pose>
+      <publish_sensor_pose>true</publish_sensor_pose>
+      <publish_collision_pose>false</publish_collision_pose>
+      <use_pose_vector_msg>true</use_pose_vector_msg>
+    </plugin>
+  </gazebo> -->
 </robot>

Commit message: updating

File: fws_description/gazebo/fws_robot.gazebo.xacro (robot description, xacro)
@@ -42,38 +42,8 @@
       </sensor>
     </gazebo>
-    <!-- GPS Link and Joint -->
-    <link name="gps_link">
-      <visual>
-        <geometry>
-          <sphere radius="0.01"/>
-        </geometry>
-        <material name="white"/>
-      </visual>
-    </link>
-    <joint name="gps_joint" type="fixed">
-      <parent link="base_link"/>
-      <child link="gps_link"/>
-      <origin xyz="0 0 0.1" rpy="0 0 0"/>
-    </joint>
-    <!-- GPS Sensor Plugin -->
-    <gazebo reference="gps_link">
-      <sensor name="gps_sensor" type="navsat">
-        <pose>0 0 0 0 0 0</pose>
-        <update_rate>5.0</update_rate>
-        <navsat>
-          <horizontal>
-            <noise type="gaussian">
-              <mean>0</mean>
-              <stddev>1e-6</stddev>
-            </noise>
-          </horizontal>
-          <vertical>
-            <noise type="gaussian">
-              <mean>0</mean>
-              <stddev>1e-6</stddev>
-            </noise>
-          </vertical>
-        </navsat>
-      </sensor>
+    <gazebo>
+      <plugin filename="gz-sim-navsat-system"
+          name="gz::sim::systems::NavSat">
+      </plugin>
     </gazebo>
   </xacro:macro>

File: fws_description/robots/fws_robot.urdf.xacro (robot description, xacro)
@@ -91,11 +91,3 @@
   <xacro:fws_robot_gazebo/>
   <xacro:fws_robot_ros2_control/>
-  <!-- <gazebo>
-  <plugin name="gz::sim::systems::PosePublisher" filename="gz-sim-pose-publisher-system">
-      <publish_link_pose>true</publish_link_pose>
-      <publish_sensor_pose>true</publish_sensor_pose>
-      <publish_collision_pose>false</publish_collision_pose>
-      <use_pose_vector_msg>true</use_pose_vector_msg>
-    </plugin>
-  </gazebo> -->
 </robot>

File: fws_description/robots/parts/base/base.urdf.xacro (robot description, xacro)
@@ -25,4 +25,42 @@
 	  </inertial>
 	</link>
+    <!-- GPS Link -->
+    <link name="gps_link">
+      <inertial>
+        <origin xyz="0 0 0"/>
+        <mass value="0.01"/>
+        <inertia ixx="1e-5" ixy="0" ixz="0" iyy="1e-5" iyz="0" izz="1e-5"/>
+      </inertial>
+    </link>
+    <!-- Joint to attach GPS to base -->
+    <joint name="gps_joint" type="fixed">
+      <parent link="base_link"/>
+      <child link="gps_link"/>
+      <origin xyz="0 0 0.5" rpy="0 0 0"/>
+    </joint>
+    <!-- Gazebo plugin for GPS -->
+    <gazebo reference="gps_link">
+      <sensor name="gps_sensor" type="gps">
+        <always_on>true</always_on>
+        <update_rate>5</update_rate>
+        <gps>
+          <position_sensing>
+            <horizontal>
+              <noise type="gaussian">
+                <mean>0.0</mean>
+                <stddev>0.0</stddev>
+              </noise>
+            </horizontal>
+            <vertical>
+              <noise type="gaussian">
+                <mean>0.0</mean>
+                <stddev>0.0</stddev>
+              </noise>
+            </vertical>
+          </position_sensing>
+        </gps>
+        <visualize>false</visualize>
+      </sensor>
+    </gazebo>
   </xacro:macro>
 </robot>

Commit message: updating sensor fusion and ADAS

File: fws_description/gazebo/fws_robot.gazebo.xacro (robot description, xacro)
@@ -47,4 +47,10 @@
       </plugin>
     </gazebo>
+    <gazebo>
+      <plugin
+        filename="gz-sim-imu-system"
+        name="gz::sim::systems::Imu">
+      </plugin>
+    </gazebo>
   </xacro:macro>
 </robot>

File: fws_description/robots/parts/base/base.urdf.xacro (robot description, xacro)
@@ -63,4 +63,28 @@
       </sensor>
     </gazebo>
+    <!-- IMU Link -->
+    <link name="imu_link">
+      <inertial>
+        <origin xyz="0 0 0"/>
+        <mass value="0.01"/>
+        <inertia ixx="1e-5" ixy="0" ixz="0" iyy="1e-5" iyz="0" izz="1e-5"/>
+      </inertial>
+    </link>
+      <!-- Joint to attach IMU to base -->
+    <joint name="imu_joint" type="fixed">
+      <parent link="base_link"/>
+      <child link="imu_link"/>
+      <origin xyz="0 0 0.05" rpy="0 0 0"/>
+    </joint>
+    <!-- Gazebo plugin for IMU -->
+    <gazebo reference="imu_link">
+      <sensor name="imu" type="imu">
+          <always_on>1</always_on>
+          <update_rate>100</update_rate>
+          <visualize>true</visualize>
+          <topic>imu</topic>
+          <enable_metrics>true</enable_metrics>
+      </sensor>
+    </gazebo>
   </xacro:macro>
 </robot>
